Commit message: Add some colors to my_robot

File: src/my_robot/urdf/my_robot.xacro (robot description, xacro)
@@ -109,4 +109,7 @@
         <cylinder radius="0.1" length="0.05" />
       </geometry>
+      <material name="black">
+        <color rgba="0.1 0.1 0.1 1.0"/>
+      </material>
     </visual>
   </link>
@@ -132,4 +135,7 @@
         <cylinder radius="0.1" length="0.05" />
       </geometry>
+      <material name="black">
+        <color rgba="0.1 0.1 0.1 1.0"/>
+      </material>
     </visual>
   </link>
@@ -145,5 +151,5 @@
       />
     </inertial>
-    <collision name='collision'>
+    <collision name='chassis_collision'>
       <origin xyz="0 0 0" rpy=" 0 0 0"/>
       <geometry>
@@ -156,4 +162,7 @@
         <box size=".4 .2 .1"/>
       </geometry>
+      <material name="metal">
+        <color rgba="0.8 0.8 0.8 1.0"/>
+      </material>
     </visual>
     <collision name='back_caster_collision'>
@@ -168,4 +177,7 @@
         <sphere radius="0.05"/>
       </geometry>
+      <material name="black">
+        <color rgba="0.1 0.1 0.1 1.0"/>
+      </material>
     </visual>
     <collision name='front_caster_collision'>
@@ -180,4 +192,7 @@
         <sphere radius="0.05"/>
       </geometry>
+      <material name="black">
+        <color rgba="0.1 0.1 0.1 1.0"/>
+      </material>
     </visual>
   </link>

Commit message: Make some collision and visual changes to my robot

File: src/my_robot/urdf/my_robot.xacro (robot description, xacro)
@@ -101,5 +101,5 @@
       <origin xyz="0 0 0" rpy="0 1.5707 1.5707"/>
       <geometry>
-        <cylinder radius="0.1" length="0.05" />
+        <cylinder radius="0.1" length="0.15" />
       </geometry>
     </collision>
@@ -107,5 +107,5 @@
       <origin xyz="0 0 0" rpy="0 1.5707 1.5707"/>
       <geometry>
-        <cylinder radius="0.1" length="0.05" />
+        <cylinder radius="0.1" length="0.15" />
       </geometry>
       <material name="black">
@@ -127,5 +127,5 @@
       <origin xyz="0.0 0 0" rpy="0 1.5707 1.5707"/>
       <geometry>
-        <cylinder radius="0.1" length="0.05" />
+        <cylinder radius="0.1" length="0.15" />
       </geometry>
     </collision>
@@ -133,5 +133,5 @@
       <origin xyz="0.0 0 0" rpy="0 1.5707 1.5707"/>
       <geometry>
-        <cylinder radius="0.1" length="0.05" />
+        <cylinder radius="0.1" length="0.15" />
       </geometry>
       <material name="black">
@@ -154,5 +154,5 @@
       <origin xyz="0 0 0" rpy=" 0 0 0"/>
       <geometry>
-        <box size=".4 .2 .1"/>
+        <box size=".4 .1 .1"/>
       </geometry>
     </collision>
@@ -160,5 +160,5 @@
       <origin xyz="0 0 0" rpy=" 0 0 0"/>
       <geometry>
-        <box size=".4 .2 .1"/>
+        <box size=".4 .1 .1"/>
       </geometry>
       <material name="metal">
