Commit message: Add mapping launch file

File: my_robot/urdf/my_robot.xacro (robot description, xacro)
@@ -26,5 +26,5 @@
   <joint type="fixed" name="camera_joint">
     <origin xyz="0.2 0 0" rpy="0 0 0"/>
-    <child link="camera"/>
+    <child link="camera_link"/>
     <parent link="chassis"/>
     <axis xyz="0 1 0" rpy="0 0 0"/>
@@ -62,5 +62,5 @@
     </visual>
   </link>
-  <link name="camera">
+  <link name="camera_link">
     <inertial>
       <mass value="0.1"/>
@@ -88,4 +88,11 @@
     </visual>
   </link>
+ <joint name="camera_optical_joint" type="fixed">
+    <origin xyz="0 0 0" rpy="-1.5707 0 -1.5707"/>
+    <parent link="camera_link"/>
+    <child link="camera_link_optical"/>
+  </joint>
+  <link name="camera_link_optical">
+  </link>
   <link name="left_wheel">
     <inertial>
